Commit message: Fixed package-naming reference and added robot-spawn launch-file

File: multi_robot_spawn/urdf/scene_urdf.xacro (robot description, xacro)
@@ -55,8 +55,8 @@
         <xacro:unless value="${robot1_eoat}">
             <!-- Robot Tool-Center-Point -->
-            <link name="$(arg robot1_prefix)tcp"/>
-            <joint name="$(arg robot1_prefix)tcp_joint" type="fixed">
+            <link name="$(arg robot1_prefix)eoat_tcp"/>
+            <joint name="$(arg robot1_prefix)eoat_tcp_joint" type="fixed">
                 <parent link="$(arg robot1_prefix)tool0"/>
-                <child link="$(arg robot1_prefix)tcp"/>
+                <child link="$(arg robot1_prefix)eoat_tcp"/>
                 <origin xyz="0.000 0.000 0.000" rpy="0.0 0.0 0.0"/>
             </joint>
@@ -114,8 +114,8 @@
         <xacro:unless value="${robot2_eoat}">
             <!-- Robot Tool-Center-Point -->
-            <link name="$(arg robot2_prefix)tcp"/>
-            <joint name="$(arg robot2_prefix)tcp_joint" type="fixed">
+            <link name="$(arg robot2_prefix)eoat_tcp"/>
+            <joint name="$(arg robot2_prefix)eoat_tcp_joint" type="fixed">
                 <parent link="$(arg robot2_prefix)tool0"/>
-                <child link="$(arg robot2_prefix)tcp"/>
+                <child link="$(arg robot2_prefix)eoat_tcp"/>
                 <origin xyz="0.000 0.000 0.000" rpy="0.0 0.0 0.0"/>
             </joint>

File: robot_spawn/urdf/scene_urdf.xacro (robot description, xacro)
@@ -43,8 +43,8 @@
     <xacro:unless value="${robot_eoat}">
         <!-- Robot Tool-Center-Point -->
-        <link name="$(arg robot_prefix)tcp"/>
-        <joint name="$(arg robot_prefix)tcp_joint" type="fixed">
+        <link name="$(arg robot_prefix)eoat_tcp"/>
+        <joint name="$(arg robot_prefix)eoat_tcp_joint" type="fixed">
             <parent link="$(arg robot_prefix)tool0"/>
-            <child link="$(arg robot_prefix)tcp"/>
+            <child link="$(arg robot_prefix)eoat_tcp"/>
             <origin xyz="0.000 0.000 0.000" rpy="0.0 0.0 0.0"/>
         </joint>
@@ -56,4 +56,4 @@
         <link name="$(arg global_ref_frame)"/>
         <!-- Environment URDF -->
-        <!-- <xacro:include filename="$(find robot_support)/urdf/environment_urdf.xacro"/> -->
+        <xacro:include filename="$(find robot_support)/urdf/environment_urdf.xacro"/>
 </robot>
